File: reflow-oven-nano-shield.sch (KiCad schematic (older format))
At the start: 41 parts, among them J1 POWER IN, J2 SSR OUT, J3 SERVO, Q1 2N3904, Q2 2N3904, Q3 2N3904, Q4 2N3904, Q5 2N3904, SW1 TOP, SW2 BOTTOM

Commit message: Hand solder TO-92 footprint, add teardrops
Parts:
- C1: value 220uf -> 1000uf; footprint Capacitor_THT:CP_Radial_D5.0mm_P2.00mm -> Capacitor_THT:CP_Radial_D8.0mm_P3.50mm
- Q1, Q2, Q3, Q4, Q5: footprint Package_TO_SOT_THT:TO-92_Inline -> Package_TO_SOT_THT:TO-92_HandSolder
Changed lines of the file:
@@
 F 0 "Q1" H 8540 1646 50  0000 L CNN
 F 1 "2N3904" H 8540 1555 50  0000 L CNN
-F 2 "Package_TO_SOT_THT:TO-92_Inline" H 8550 1525 50  0001 L CIN
+F 2 "Package_TO_SOT_THT:TO-92_HandSolder" H 8550 1525 50  0001 L CIN
 F 3 "https://www.onsemi.com/pub/Collateral/2N3903-D.PDF" H 8350 1600 50  0001 L CNN
 	1    8350 1600
@@
 F 0 "Q2" H 8540 3296 50  0000 L CNN
 F 1 "2N3904" H 8540 3205 50  0000 L CNN
-F 2 "Package_TO_SOT_THT:TO-92_Inline" H 8550 3175 50  0001 L CIN
+F 2 "Package_TO_SOT_THT:TO-92_HandSolder" H 8550 3175 50  0001 L CIN
 F 3 "https://www.onsemi.com/pub/Collateral/2N3903-D.PDF" H 8350 3250 50  0001 L CNN
 	1    8350 3250
@@
 F 0 "Q4" H 10040 1646 50  0000 L CNN
 F 1 "2N3904" H 10040 1555 50  0000 L CNN
-F 2 "Package_TO_SOT_THT:TO-92_Inline" H 10050 1525 50  0001 L CIN
+F 2 "Package_TO_SOT_THT:TO-92_HandSolder" H 10050 1525 50  0001 L CIN
 F 3 "https://www.onsemi.com/pub/Collateral/2N3903-D.PDF" H 9850 1600 50  0001 L CNN
 	1    9850 1600
@@
 F 0 "Q3" H 9240 4796 50  0000 L CNN
 F 1 "2N3904" H 9240 4705 50  0000 L CNN
-F 2 "Package_TO_SOT_THT:TO-92_Inline" H 9250 4675 50  0001 L CIN
+F 2 "Package_TO_SOT_THT:TO-92_HandSolder" H 9250 4675 50  0001 L CIN
 F 3 "https://www.onsemi.com/pub/Collateral/2N3903-D.PDF" H 9050 4750 50  0001 L CNN
 	1    9050 4750
@@
 F 0 "Q5" H 10040 3296 50  0000 L CNN
 F 1 "2N3904" H 10040 3205 50  0000 L CNN
-F 2 "Package_TO_SOT_THT:TO-92_Inline" H 10050 3175 50  0001 L CIN
+F 2 "Package_TO_SOT_THT:TO-92_HandSolder" H 10050 3175 50  0001 L CIN
 F 3 "https://www.onsemi.com/pub/Collateral/2N3903-D.PDF" H 9850 3250 50  0001 L CNN
 	1    9850 3250
@@
 P 1100 5650
 F 0 "C1" H 985 5604 50  0000 R CNN
-F 1 "220uf" H 985 5695 50  0000 R CNN
-F 2 "Capacitor_THT:CP_Radial_D5.0mm_P2.00mm" H 1100 5650 50  0001 C CNN
+F 1 "1000uf" H 985 5695 50  0000 R CNN
+F 2 "Capacitor_THT:CP_Radial_D8.0mm_P3.50mm" H 1100 5650 50  0001 C CNN
 F 3 "~" H 1100 5650 50  0001 C CNN
 	1    1100 5650
